File: cpu_interface.kicad_sch (KiCad schematic)
At the start: 21 parts, among them J111 J111 G.I. latch spare bits T5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, J113 34-pin ribbon to CPU J211, U6 LM339DR, U9 74HCT240

Commit message: Prepare WPC engineering candidate and verification tooling
Include revised PCB and schematics, component models, fabrication exports, renders, BOM, assembly counts, and reproducible electrical and manufacturing checks. Document unresolved replay convergence, regulator fault behavior, and physical qualification gates; this candidate is not production released.
Parts:
- B6, B9: symbol Device:C -> wpc_symbols:Device_C
- C21: symbol Device:C -> wpc_symbols:Device_C; Link https://www.digikey.com/en/products/result?keywords=CL21B10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 -> https://search.kemet.com/download/specsheet/C0805C103K5RACTU; MPN CL21B103KBANNNC -> C0805C103K5RACTU; Manufacturer Samsung -> KEMET
- J111: symbol Connector_Generic:Conn_01x05 -> wpc_symbols:Connector_Generic_Conn_01x05
- J113: footprint Connector_IDC:IDC-Header_2x17_P2.54mm_Vertical -> wpc_cost:3M_N2534_6002_RB; symbol Connector_Generic:Conn_02x17_Odd_Even -> wpc_symbols:Connector_Generic_Conn_02x17_Odd_Even; Link https://www.digikey.com/en/products/detail/3m/30334-5002HB/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 -> https://www.digikey.com/en/products/detail/3m/N2534-6002-RB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; MPN 30334-5002HB -> N2534-6002-RB
- LED3: symbol Device:LED -> wpc_symbols:Device_LED
- R197, R198, R206, R253, R254, R255, R256, R3, R4, R6: symbol Device:R -> wpc_symbols:Device_R
- SR1, SR2: symbol Device:R_Network09 -> wpc_symbols:Device_R_Network09
- TP4: symbol Connector:TestPoint -> wpc_symbols:Connector_TestPoint
- U6: symbol Comparator:LM339 -> wpc_symbols:Comparator_LM339
- U9: symbol 74xx:74HCT240 -> wpc_symbols:74xx_74HCT240
Changed lines of the file:
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@@
 	)
 	(symbol
-		(lib_id "Connector_Generic:Conn_02x17_Odd_Even")
+		(lib_id "wpc_symbols:Connector_Generic_Conn_02x17_Odd_Even")
 		(at 59.69 100.33 0)
 		(unit 1)
@@
 			)
 		)
-		(property "Footprint" "Connector_IDC:IDC-Header_2x17_P2.54mm_Vertical"
+		(property "Footprint" "wpc_cost:3M_N2534_6002_RB"
 			(at 59.69 100.33 0)
 			(effects
@@
 			)
 		)
-		(property "MPN" "30334-5002HB"
+		(property "MPN" "N2534-6002-RB"
 			(at 59.69 100.33 0)
 			(effects
@@
 			)
 		)
-		(property "Link" "https://www.digikey.com/en/products/detail/3m/30334-5002HB/1237402"
+		(property "Link" "https://www.digikey.com/en/products/detail/3m/N2534-6002-RB/755183"
 			(at 59.69 100.33 0)
 			(effects
@@
 	)
 	(symbol
-		(lib_id "power:GND")
+		(lib_id "wpc_symbols:power_GND")
 		(at 72.39 82.55 0)
 		(unit 1)
@@
 	)
 	(symbol
-		(lib_id "power:GND")
+		(lib_id "wpc_symbols:power_GND")
 		(at 72.39 85.09 0)
 		(unit 1)
@@
 	)
 	(symbol
-		(lib_id "power:GND")
+		(lib_id "wpc_symbols:power_GND")
 		(at 72.39 95.25 0)
 		(unit 1)
@@
 	)
 	(symbol
-		(lib_id "power:GND")
+		(lib_id "wpc_symbols:power_GND")
 		(at 72.39 97.79 0)
 		(unit 1)
@@
 	)
 	(symbol
-		(lib_id "power:GND")
+		(lib_id "wpc_symbols:power_GND")
 		(at 72.39 100.33 0)
 		(unit 1)
@@
 	)
 	(symbol
-		(lib_id "power:GND")
+		(lib_id "wpc_symbols:power_GND")
 		(at 72.39 102.87 0)
 		(unit 1)
@@
 	)
 	(symbol
-		(lib_id "power:GND")
+		(lib_id "wpc_symbols:power_GND")
 		(at 72.39 105.41 0)
 		(unit 1)
@@
 	)
 	(symbol
-		(lib_id "power:GND")
+		(lib_id "wpc_symbols:power_GND")
 		(at 72.39 107.95 0)
 		(unit 1)
@@
 	)
 	(symbol
-		(lib_id "power:GND")
+		(lib_id "wpc_symbols:power_GND")
 		(at 72.39 110.49 0)
 		(unit 1)
@@
 	)
 	(symbol
-		(lib_id "power:GND")
+		(lib_id "wpc_symbols:power_GND")
 		(at 72.39 113.03 0)
 		(unit 1)
@@
 	)
 	(symbol
-		(lib_id "power:GND")
+		(lib_id "wpc_symbols:power_GND")
 		(at 72.39 115.57 0)
 		(unit 1)
@@
 	)
 	(symbol
-		(lib_id "74xx:74HCT240")
+		(lib_id "wpc_symbols:74xx_74HCT240")
 		(at 170.18 100.33 0)
 		(unit 1)
@@
 	)
 	(symbol
-		(lib_id "power:GND")
+		(lib_id "wpc_symbols:power_GND")
 		(at 152.4 110.49 0)
 		(unit 1)
@@
 	)
 	(symbol
-		(lib_id "power:GND")
+		(lib_id "wpc_symbols:power_GND")
 		(at 152.4 113.03 0)
 		(unit 1)
@@
 	)
 	(symbol
-		(lib_id "power:+5V")
+		(lib_id "wpc_symbols:power_+5V")
 		(at 170.18 80.01 0)
 		(unit 1)
@@
 	)
 	(symbol
-		(lib_id "power:GND")
+		(lib_id "wpc_symbols:power_GND")
 		(at 170.18 120.65 0)
 		(unit 1)
@@
 	)
 	(symbol
-		(lib_id "Device:C")
+		(lib_id "wpc_symbols:Device_C")
 		(at 234.95 110.49 0)
 		(unit 1)
@@
 	)
 	(symbol
-		(lib_id "power:+5V")
+		(lib_id "wpc_symbols:power_+5V")
 		(at 234.95 106.68 0)
 		(unit 1)
@@
 	)
 	(symbol
-		(lib_id "power:GND")
+		(lib_id "wpc_symbols:power_GND")
 		(at 234.95 114.3 0)
 		(unit 1)
@@
 	)
 	(symbol
-		(lib_id "Device:R_Network09")
+		(lib_id "wpc_symbols:Device_R_Network09")
 		(at 214.63 39.37 0)
 		(unit 1)
@@
 	)
 	(symbol
-		(lib_id "power:+5V")
+		(lib_id "wpc_symbols:power_+5V")
 		(at 204.47 34.29 0)
 		(unit 1)
@@
 	)
 	(symbol
-		(lib_id "Device:R_Network09")
+		(lib_id "wpc_symbols:Device_R_Network09")
 		(at 255.27 39.37 0)
 		(unit 1)
@@
 	)
 	(symbol
-		(lib_id "power:+5V")
+		(lib_id "wpc_symbols:power_+5V")
 		(at 245.11 34.29 0)
 		(unit 1)
@@
 	)
 	(symbol
-		(lib_id "Device:C")
+		(lib_id "wpc_symbols:Device_C")
 		(at 214.63 110.49 0)
 		(unit 1)
@@
 	)
 	(symbol
-		(lib_id "power:+5V")
+		(lib_id "wpc_symbols:power_+5V")
 		(at 214.63 106.68 0)
 		(unit 1)
@@
 	)
 	(symbol
-		(lib_id "power:GND")
+		(lib_id "wpc_symbols:power_GND")
 		(at 214.63 114.3 0)
 		(unit 1)
@@
 	)
 	(symbol
-		(lib_id "Device:R")
+		(lib_id "wpc_symbols:Device_R")
 		(at 269.24 80.01 90)
 		(unit 1)
@@
 	)
 	(symbol
-		(lib_id "Device:R")
+		(lib_id "wpc_symbols:Device_R")
 		(at 269.24 87.63 90)
 		(unit 1)
@@
 	)
 	(symbol
-		(lib_id "Device:R")
+		(lib_id "wpc_symbols:Device_R")
 		(at 279.4 90.17 0)
 		(unit 1)
@@
 	)
 	(symbol
-		(lib_id "Comparator:LM339")
+		(lib_id "wpc_symbols:Comparator_LM339")
 		(at 299.72 82.55 0)
 		(unit 1)
@@
 	)
 	(symbol
-		(lib_id "Device:R")
+		(lib_id "wpc_symbols:Device_R")
 		(at 312.42 74.93 0)
 		(unit 1)
@@
 	)
 	(symbol
-		(lib_id "Device:R")
+		(lib_id "wpc_symbols:Device_R")
 		(at 279.4 67.31 0)
 		(unit 1)
@@
 	)
 	(symbol
-		(lib_id "Device:R")
+		(lib_id "wpc_symbols:Device_R")
 		(at 279.4 77.47 0)
 		(unit 1)
@@
 	)
 	(symbol
-		(lib_id "Device:C")
+		(lib_id "wpc_symbols:Device_C")
 		(at 287.02 90.17 0)
 		(unit 1)
@@
 			)
 		)
-		(property "MPN" "CL21B103KBANNNC"
+		(property "MPN" "C0805C103K5RACTU"
 			(at 287.02 90.17 0)
 			(effects
@@
 			)
 		)
-		(property "Manufacturer" "Samsung"
+		(property "Manufacturer" "KEMET"
 			(at 287.02 90.17 0)
 			(effects
@@
 			)
 		)
-		(property "Link" "https://www.digikey.com/en/products/result?keywords=CL21B103KBANNNC"
+		(property "Link" "https://search.kemet.com/download/specsheet/C0805C103K5RACTU"
 			(at 287.02 90.17 0)
 			(effects
@@
 	)
 	(symbol
-		(lib_id "power:GND")
+		(lib_id "wpc_symbols:power_GND")
 		(at 279.4 93.98 0)
 		(unit 1)
@@
 	)
 	(symbol
-		(lib_id "power:GND")
+		(lib_id "wpc_symbols:power_GND")
 		(at 287.02 93.98 0)
 		(unit 1)
@@
 	)
 	(symbol
-		(lib_id "power:+5V")
+		(lib_id "wpc_symbols:power_+5V")
 		(at 279.4 63.5 0)
 		(unit 1)
@@
 	)
 	(symbol
-		(lib_id "power:GND")
+		(lib_id "wpc_symbols:power_GND")
 		(at 279.4 81.28 0)
 		(unit 1)
@@
 	)
 	(symbol
-		(lib_id "power:+5V")
+		(lib_id "wpc_symbols:power_+5V")
 		(at 312.42 71.12 0)
 		(unit 1)
@@
 	)
 	(symbol
-		(lib_id "Connector:TestPoint")
+		(lib_id "wpc_symbols:Connector_TestPoint")
 		(at 314.96 77.47 0)
 		(unit 1)
@@
 	)
 	(symbol
-		(lib_id "Device:R")
+		(lib_id "wpc_symbols:Device_R")
 		(at 330.2 82.55 90)
 		(unit 1)
@@
 	)
 	(symbol
-		(lib_id "Device:LED")
+		(lib_id "wpc_symbols:Device_LED")
 		(at 341.63 82.55 0)
 		(unit 1)
@@
 	)
 	(symbol
-		(lib_id "power:+5V")
+		(lib_id "wpc_symbols:power_+5V")
 		(at 345.44 82.55 0)
 		(unit 1)
@@
 	)
 	(symbol
-		(lib_id "Comparator:LM339")
+		(lib_id "wpc_symbols:Comparator_LM339")
 		(at 299.72 119.38 0)
 		(unit 2)
@@
 	)
 	(symbol
-		(lib_id "Device:R")
+		(lib_id "wpc_symbols:Device_R")
 		(at 279.4 106.68 0)
 		(unit 1)
@@
 	)
 	(symbol
-		(lib_id "Device:R")
+		(lib_id "wpc_symbols:Device_R")
 		(at 279.4 116.84 0)
 		(unit 1)
@@
 	)
 	(symbol
-		(lib_id "Device:R")
+		(lib_id "wpc_symbols:Device_R")
 		(at 269.24 121.92 90)
 		(unit 1)
@@
 	)
 	(symbol
-		(lib_id "power:+5V")
+		(lib_id "wpc_symbols:power_+5V")
 		(at 279.4 102.87 0)
 		(unit 1)
@@
 	)
 	(symbol
-		(lib_id "power:GND")
+		(lib_id "wpc_symbols:power_GND")
 		(at 279.4 120.65 0)
 		(unit 1)
@@
 	)
 	(symbol
-		(lib_id "Comparator:LM339")
+		(lib_id "wpc_symbols:Comparator_LM339")
 		(at 299.72 144.78 0)
 		(unit 3)
@@
 	)
 	(symbol
-		(lib_id "power:GND")
+		(lib_id "wpc_symbols:power_GND")
 		(at 292.1 142.24 0)
 		(unit 1)
@@
 	)
 	(symbol
-		(lib_id "power:+5V")
+		(lib_id "wpc_symbols:power_+5V")
 		(at 289.56 147.32 0)
 		(unit 1)
@@
 	)
 	(symbol
-		(lib_id "Comparator:LM339")
+		(lib_id "wpc_symbols:Comparator_LM339")
 		(at 299.72 165.1 0)
 		(unit 4)
@@
 	)
 	(symbol
-		(lib_id "power:GND")
+		(lib_id "wpc_symbols:power_GND")
 		(at 292.1 162.56 0)
 		(unit 1)
@@
 	)
 	(symbol
-		(lib_id "power:+5V")
+		(lib_id "wpc_symbols:power_+5V")
 		(at 289.56 167.64 0)
 		(unit 1)
@@
 	)
 	(symbol
-		(lib_id "Comparator:LM339")
+		(lib_id "wpc_symbols:Comparator_LM339")
 		(at 359.41 149.86 0)
 		(unit 5)
@@
 	)
 	(symbol
-		(lib_id "power:+5V")
+		(lib_id "wpc_symbols:power_+5V")
 		(at 356.87 142.24 0)
 		(unit 1)
@@
 	)
 	(symbol
-		(lib_id "power:GND")
+		(lib_id "wpc_symbols:power_GND")
 		(at 356.87 157.48 0)
 		(unit 1)
@@
 	)
 	(symbol
-		(lib_id "Connector_Generic:Conn_01x05")
+		(lib_id "wpc_symbols:Connector_Generic_Conn_01x05")
 		(at 384.81 59.69 0)
 		(unit 1)
@@
 	)
 	(symbol
-		(lib_id "power:GND")
+		(lib_id "wpc_symbols:power_GND")
 		(at 374.65 64.77 0)
 		(unit 1)
