File: gi_triacs.kicad_sch (KiCad schematic)
At the start: 45 parts, among them J105 J105 fused 51VAC (F112, pins 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, J115 J115 G.I. 6.3VAC from transfo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, J119 J119 G.I. coin door (string 5), J120 J120 G.I. strings 1-5 (backbo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, J121 J121 G.I. strings 1-5 (playfi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, Q10 BTA16-600CRG, Q11 MMBT4401, Q12 BTA16-600CRG, Q13 MMBT4401, Q14 BTA16-600CRG, Q15 MMBT4401, Q16 BTA16-600CRG, Q17 MMBT4401, Q18 BTA16-600CRG, Q3 IRLR3110ZTRPBF (DNP), Q9 MMBT4401, U1 74HCT574

Commit message: Prepare WPC engineering candidate and verification tooling
Include revised PCB and schematics, component models, fabrication exports, renders, BOM, assembly counts, and reproducible electrical and manufacturing checks. Document unresolved replay convergence, regulator fault behavior, and physical qualification gates; this candidate is not production released.
Parts:
- B1: symbol Device:C -> wpc_symbols:Device_C
- D35: symbol Diode:1N4007 -> wpc_symbols:Diode_1N4007
- F101, F102, F106, F107, F108, F109, F110: symbol Device:Fuse -> wpc_symbols:Device_Fuse
- J105: symbol Connector_Generic:Conn_01x05 -> wpc_symbols:Connector_Generic_Conn_01x05; Link https://www.digikey.com/en/products/result?keywords=0026604005 -> https://www.digikey.com/en/products/result?keywords=0026604050; MPN 0026604005 -> 0026604050
- J115: symbol Connector_Generic:Conn_01x12 -> wpc_symbols:Connector_Generic_Conn_01x12; Link https://www.digikey.com/en/products/result?keywords=0026604012 -> https://www.digikey.com/en/products/result?keywords=0026604120; MPN 0026604012 -> 0026604120
- J119: symbol Connector_Generic:Conn_01x03 -> wpc_symbols:Connector_Generic_Conn_01x03; Link https://www.digikey.com/en/products/result?keywords=0026604003 -> https://www.digikey.com/en/products/result?keywords=0026604030; MPN 0026604003 -> 0026604030
- J120, J121: symbol Connector_Generic:Conn_01x11 -> wpc_symbols:Connector_Generic_Conn_01x11; Link https://www.digikey.com/en/products/result?keywords=0026604011 -> https://www.digikey.com/en/products/result?keywords=0026604110; MPN 0026604011 -> 0026604110
- Q10, Q12, Q14, Q16, Q18: symbol Triac_Thyristor:BTA16-600C -> wpc_symbols:Triac_Thyristor_BTA16-600C
- Q11, Q13, Q15, Q17, Q9: symbol Transistor_BJT:Q_NPN_BEC -> wpc_symbols:Transistor_BJT_Q_NPN_BEC
- Q3: value IRLR3110ZTRPBF (DNP) -> IPD90N10S4L06ATMA1; symbol Transistor_FET:Q_NMOS_GDS -> wpc_symbols:Transistor_FET_Q_NMOS_GDS; Link https://www.digikey.com/en/products/detail/infineon-technol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 -> https://www.infineon.com/part/IPD90N10S4L-06; MPN IRLR3110ZTRPBF -> IPD90N10S4L06ATMA1
- R10, R11, R12, R13, R14, R15, R16, R17, R18, R19, R20, R202, R209, R21, R7, R8, R9, W1: symbol Device:R -> wpc_symbols:Device_R
- RLY1: symbol Relay:G2RL-2 -> wpc_symbols:Relay_G2RL-2
- U1: symbol 74xx:74HCT574 -> wpc_symbols:74xx_74HCT574
