File: lamp_columns.kicad_sch (KiCad schematic)
At the start: 31 parts, among them J136 J136 lamp column 8 (cabinet), J137 J137 lamp columns (playfield), J138 J138 lamp columns (backbox), Q91 IRFR5305TRPBF, Q92 IRFR5305TRPBF, Q93 IRFR5305TRPBF, Q94 IRFR5305TRPBF, Q95 IRFR5305TRPBF, Q96 IRFR5305TRPBF, Q97 IRFR5305TRPBF, Q98 IRFR5305TRPBF, U18 74HCT574, U19 TBD62083AFWG

Commit message: Prepare WPC engineering candidate and verification tooling
Include revised PCB and schematics, component models, fabrication exports, renders, BOM, assembly counts, and reproducible electrical and manufacturing checks. Document unresolved replay convergence, regulator fault behavior, and physical qualification gates; this candidate is not production released.
Parts:
- B18, B19: symbol Device:C -> wpc_symbols:Device_C
- J136: symbol Connector_Generic:Conn_01x03 -> wpc_symbols:Connector_Generic_Conn_01x03; Link https://www.digikey.com/en/products/result?keywords=0026604003 -> https://www.digikey.com/en/products/result?keywords=0026604030; MPN 0026604003 -> 0026604030
- J137, J138: symbol Connector_Generic:Conn_01x09 -> wpc_symbols:Connector_Generic_Conn_01x09; MPN 0026604009 -> 0026604090
- Q91, Q92, Q93, Q94, Q95, Q96, Q97, Q98: symbol Transistor_FET:Q_PMOS_GDS -> wpc_symbols:Transistor_FET_Q_PMOS_GDS
- R176, R177, R178, R179, R180, R181, R182, R183, R184, R185, R186, R187, R188, R189, R190, R191: symbol Device:R -> wpc_symbols:Device_R
- U18: symbol 74xx:74HCT574 -> wpc_symbols:74xx_74HCT574
- U19: symbol Transistor_Array:ULN2803A -> wpc_symbols:Transistor_Array_ULN2803A
Changed lines of the file:
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@@
 	)
 	(symbol
-		(lib_id "Transistor_FET:Q_PMOS_GDS")
+		(lib_id "wpc_symbols:Transistor_FET_Q_PMOS_GDS")
 		(at 80.01 59.69 0)
 		(mirror x)
@@
 	)
 	(symbol
-		(lib_id "Device:R")
+		(lib_id "wpc_symbols:Device_R")
 		(at 74.93 52.07 0)
 		(unit 1)
@@
 	)
 	(symbol
-		(lib_id "Device:R")
+		(lib_id "wpc_symbols:Device_R")
 		(at 67.31 59.69 90)
 		(unit 1)
@@
 	)
 	(symbol
-		(lib_id "power:+18V")
+		(lib_id "wpc_symbols:wpc_power_+18V")
 		(at 82.55 46.99 0)
 		(unit 1)
@@
 	)
 	(symbol
-		(lib_id "Transistor_FET:Q_PMOS_GDS")
+		(lib_id "wpc_symbols:Transistor_FET_Q_PMOS_GDS")
 		(at 149.86 59.69 0)
 		(mirror x)
@@
 	)
 	(symbol
-		(lib_id "Device:R")
+		(lib_id "wpc_symbols:Device_R")
 		(at 144.78 52.07 0)
 		(unit 1)
@@
 	)
 	(symbol
-		(lib_id "Device:R")
+		(lib_id "wpc_symbols:Device_R")
 		(at 137.16 59.69 90)
 		(unit 1)
@@
 	)
 	(symbol
-		(lib_id "power:+18V")
+		(lib_id "wpc_symbols:wpc_power_+18V")
 		(at 152.4 46.99 0)
 		(unit 1)
@@
 	)
 	(symbol
-		(lib_id "Transistor_FET:Q_PMOS_GDS")
+		(lib_id "wpc_symbols:Transistor_FET_Q_PMOS_GDS")
 		(at 219.71 59.69 0)
 		(mirror x)
@@
 	)
 	(symbol
-		(lib_id "Device:R")
+		(lib_id "wpc_symbols:Device_R")
 		(at 214.63 52.07 0)
 		(unit 1)
@@
 	)
 	(symbol
-		(lib_id "Device:R")
+		(lib_id "wpc_symbols:Device_R")
 		(at 207.01 59.69 90)
 		(unit 1)
@@
 	)
 	(symbol
-		(lib_id "power:+18V")
+		(lib_id "wpc_symbols:wpc_power_+18V")
 		(at 222.25 46.99 0)
 		(unit 1)
@@
 	)
 	(symbol
-		(lib_id "Transistor_FET:Q_PMOS_GDS")
+		(lib_id "wpc_symbols:Transistor_FET_Q_PMOS_GDS")
 		(at 289.56 59.69 0)
 		(mirror x)
@@
 	)
 	(symbol
-		(lib_id "Device:R")
+		(lib_id "wpc_symbols:Device_R")
 		(at 284.48 52.07 0)
 		(unit 1)
@@
 	)
 	(symbol
-		(lib_id "Device:R")
+		(lib_id "wpc_symbols:Device_R")
 		(at 276.86 59.69 90)
 		(unit 1)
@@
 	)
 	(symbol
-		(lib_id "power:+18V")
+		(lib_id "wpc_symbols:wpc_power_+18V")
 		(at 292.1 46.99 0)
 		(unit 1)
@@
 	)
 	(symbol
-		(lib_id "Transistor_FET:Q_PMOS_GDS")
+		(lib_id "wpc_symbols:Transistor_FET_Q_PMOS_GDS")
 		(at 80.01 115.57 0)
 		(mirror x)
@@
 	)
 	(symbol
-		(lib_id "Device:R")
+		(lib_id "wpc_symbols:Device_R")
 		(at 74.93 107.95 0)
 		(unit 1)
@@
 	)
 	(symbol
-		(lib_id "Device:R")
+		(lib_id "wpc_symbols:Device_R")
 		(at 67.31 115.57 90)
 		(unit 1)
@@
 	)
 	(symbol
-		(lib_id "power:+18V")
+		(lib_id "wpc_symbols:wpc_power_+18V")
 		(at 82.55 102.87 0)
 		(unit 1)
@@
 	)
 	(symbol
-		(lib_id "Transistor_FET:Q_PMOS_GDS")
+		(lib_id "wpc_symbols:Transistor_FET_Q_PMOS_GDS")
 		(at 149.86 115.57 0)
 		(mirror x)
@@
 	)
 	(symbol
-		(lib_id "Device:R")
+		(lib_id "wpc_symbols:Device_R")
 		(at 144.78 107.95 0)
 		(unit 1)
@@
 	)
 	(symbol
-		(lib_id "Device:R")
+		(lib_id "wpc_symbols:Device_R")
 		(at 137.16 115.57 90)
 		(unit 1)
@@
 	)
 	(symbol
-		(lib_id "power:+18V")
+		(lib_id "wpc_symbols:wpc_power_+18V")
 		(at 152.4 102.87 0)
 		(unit 1)
@@
 	)
 	(symbol
-		(lib_id "Transistor_FET:Q_PMOS_GDS")
+		(lib_id "wpc_symbols:Transistor_FET_Q_PMOS_GDS")
 		(at 219.71 115.57 0)
 		(mirror x)
@@
 	)
 	(symbol
-		(lib_id "Device:R")
+		(lib_id "wpc_symbols:Device_R")
 		(at 214.63 107.95 0)
 		(unit 1)
@@
 	)
 	(symbol
-		(lib_id "Device:R")
+		(lib_id "wpc_symbols:Device_R")
 		(at 207.01 115.57 90)
 		(unit 1)
@@
 	)
 	(symbol
-		(lib_id "power:+18V")
+		(lib_id "wpc_symbols:wpc_power_+18V")
 		(at 222.25 102.87 0)
 		(unit 1)
@@
 	)
 	(symbol
-		(lib_id "Transistor_FET:Q_PMOS_GDS")
+		(lib_id "wpc_symbols:Transistor_FET_Q_PMOS_GDS")
 		(at 289.56 115.57 0)
 		(mirror x)
@@
 	)
 	(symbol
-		(lib_id "Device:R")
+		(lib_id "wpc_symbols:Device_R")
 		(at 284.48 107.95 0)
 		(unit 1)
@@
 	)
 	(symbol
-		(lib_id "Device:R")
+		(lib_id "wpc_symbols:Device_R")
 		(at 276.86 115.57 90)
 		(unit 1)
@@
 	)
 	(symbol
-		(lib_id "power:+18V")
+		(lib_id "wpc_symbols:wpc_power_+18V")
 		(at 292.1 102.87 0)
 		(unit 1)
@@
 	)
 	(symbol
-		(lib_id "74xx:74HCT574")
+		(lib_id "wpc_symbols:74xx_74HCT574")
 		(at 59.69 199.39 0)
 		(unit 1)
@@
 	)
 	(symbol
-		(lib_id "power:+5V")
+		(lib_id "wpc_symbols:power_+5V")
 		(at 59.69 179.07 0)
 		(unit 1)
@@
 	)
 	(symbol
-		(lib_id "power:GND")
+		(lib_id "wpc_symbols:power_GND")
 		(at 59.69 219.71 0)
 		(unit 1)
@@
 	)
 	(symbol
-		(lib_id "Device:C")
+		(lib_id "wpc_symbols:Device_C")
 		(at 110.49 185.42 0)
 		(unit 1)
@@
 	)
 	(symbol
-		(lib_id "power:+5V")
+		(lib_id "wpc_symbols:power_+5V")
 		(at 110.49 181.61 0)
 		(unit 1)
@@
 	)
 	(symbol
-		(lib_id "power:GND")
+		(lib_id "wpc_symbols:power_GND")
 		(at 110.49 189.23 0)
 		(unit 1)
@@
 	)
 	(symbol
-		(lib_id "Transistor_Array:ULN2803A")
+		(lib_id "wpc_symbols:Transistor_Array_ULN2803A")
 		(at 180.34 199.39 0)
 		(unit 1)
@@
 	)
 	(symbol
-		(lib_id "power:GND")
+		(lib_id "wpc_symbols:power_GND")
 		(at 180.34 217.17 0)
 		(unit 1)
@@
 	)
 	(symbol
-		(lib_id "power:+18V")
+		(lib_id "wpc_symbols:wpc_power_+18V")
 		(at 195.58 191.77 0)
 		(unit 1)
@@
 	)
 	(symbol
-		(lib_id "Device:C")
+		(lib_id "wpc_symbols:Device_C")
 		(at 229.87 185.42 0)
 		(unit 1)
@@
 	)
 	(symbol
-		(lib_id "power:+5V")
+		(lib_id "wpc_symbols:power_+5V")
 		(at 229.87 181.61 0)
 		(unit 1)
@@
 	)
 	(symbol
-		(lib_id "power:GND")
+		(lib_id "wpc_symbols:power_GND")
 		(at 229.87 189.23 0)
 		(unit 1)
@@
 	)
 	(symbol
-		(lib_id "Connector_Generic:Conn_01x09")
+		(lib_id "wpc_symbols:Connector_Generic_Conn_01x09")
 		(at 299.72 199.39 0)
 		(unit 1)
@@
 			)
 		)
-		(property "MPN" "0026604009"
+		(property "MPN" "0026604090"
 			(at 299.72 199.39 0)
 			(effects
@@
 	)
 	(symbol
-		(lib_id "Connector_Generic:Conn_01x09")
+		(lib_id "wpc_symbols:Connector_Generic_Conn_01x09")
 		(at 359.41 199.39 0)
 		(unit 1)
@@
 			)
 		)
-		(property "MPN" "0026604009"
+		(property "MPN" "0026604090"
 			(at 359.41 199.39 0)
 			(effects
@@
 	)
 	(symbol
-		(lib_id "Connector_Generic:Conn_01x03")
+		(lib_id "wpc_symbols:Connector_Generic_Conn_01x03")
 		(at 372.11 160.02 0)
 		(unit 1)
@@
 			)
 		)
-		(property "MPN" "0026604003"
+		(property "MPN" "0026604030"
 			(at 372.11 160.02 0)
 			(effects
@@
 			)
 		)
-		(property "Link" "https://www.digikey.com/en/products/result?keywords=0026604003"
+		(property "Link" "https://www.digikey.com/en/products/result?keywords=0026604030"
 			(at 372.11 160.02 0)
 			(effects
