File: lamp_rows.kicad_sch (KiCad schematic)
At the start: 75 parts, among them J133 J133 lamp rows (cabinet), J134 J134 lamp rows (spare), J135 J135 lamp rows (playfield), Q83 IRLR024NTRPBF, Q84 IRLR024NTRPBF, Q85 IRLR024NTRPBF, Q86 IRLR024NTRPBF, Q87 IRLR024NTRPBF, Q88 IRLR024NTRPBF, Q89 IRLR024NTRPBF, Q90 IRLR024NTRPBF, U10 74HCT74, U11 74HCT74, U12 74HCT74, U13 74HCT74, U15 LM339DR, U16 LM339DR

Commit message: Prepare WPC engineering candidate and verification tooling
Include revised PCB and schematics, component models, fabrication exports, renders, BOM, assembly counts, and reproducible electrical and manufacturing checks. Document unresolved replay convergence, regulator fault behavior, and physical qualification gates; this candidate is not production released.
Parts:
- B10, B11, B12, B13, B15, B16, C13, C14, C15, C16, C17, C18, C19, C20, C31: symbol Device:C -> wpc_symbols:Device_C
- D33, D34: symbol Diode:1N4148W -> wpc_symbols:Diode_1N4148W
- J133, J134, J135: symbol Connector_Generic:Conn_01x09 -> wpc_symbols:Connector_Generic_Conn_01x09
- Q83, Q84, Q85, Q86, Q87, Q88, Q89, Q90: symbol Transistor_FET:Q_NMOS_GDS -> wpc_symbols:Transistor_FET_Q_NMOS_GDS
- R142, R143, R144, R145, R146, R147, R148, R149, R150, R151, R152, R153, R154, R155, R156, R157, R158, R159, R160, R161, R162, R164, R165, R166, R167, R168, R169, R170, R171, R172, R173, R174, R175, R301, R302, R303, R304, R305, R306, R307, R308: symbol Device:R -> wpc_symbols:Device_R
- U10, U11, U12, U13: symbol 74xx:74HCT74 -> wpc_symbols:74xx_74HCT74
- U15, U16: symbol Comparator:LM339 -> wpc_symbols:Comparator_LM339
