File: power_supply.kicad_sch (KiCad schematic)
At the start: 111 parts, among them J101 J101 xformer 9VAC (Red) / 13V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, J102 J102 xformer 16VAC (Wht-Red) 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, J103 J103 ground to 8-driver board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, J104 J104 fused 51VAC (F112, pins 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, J106 J106 +20V to backbox flashlam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, J107 J107 +50V (F103/F104/F105) an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, J108 J108 +50V (F103/F104/F105) to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, J109 J109 spare (N/C), J110 J110 spare (N/C), J112 J112 xformer 9.8VAC (Wht-Grn), J114 J114 +12V/+5V/GND to CPU J210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, J116 J116 +12V power (unregulated)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, J117 J117 +12V power (unregulated)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, J118 J118 +12V power (unregulated)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, U20 TPS54360BDDAR, U21 TPS54360BDDAR

Commit message: Prepare WPC engineering candidate and verification tooling
Include revised PCB and schematics, component models, fabrication exports, renders, BOM, assembly counts, and reproducible electrical and manufacturing checks. Document unresolved replay convergence, regulator fault behavior, and physical qualification gates; this candidate is not production released.
Parts:
- BR3: symbol Device:D_Bridge_+-AA -> wpc_symbols:Device_D_Bridge_+-AA
- C11, C30, C6, C7: value 10000uF 25V -> 10000uF 35V; footprint Capacitor_THT:CP_Radial_D25.0mm_P10.00mm_SnapIn -> Capacitor_THT:CP_Radial_D26.0mm_P10.00mm_SnapIn; symbol Device:C_Polarized -> wpc_symbols:Device_C_Polarized; Link https://www.digikey.com/en/products/detail/rubycon/25USC100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 -> https://product.tdk.com/en/search/capacitor/aluminum-electr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; MPN 25USC10000MEFCSN25X25 -> B41252A7109M000; Manufacturer Rubycon -> TDK
- C12, C2, C32, C4, C8, C9: symbol Device:C_Polarized -> wpc_symbols:Device_C_Polarized
- C33, C34, C35, C38, C39, C40, C41, C42, C44: symbol Device:C -> wpc_symbols:Device_C
- C36: symbol Device:C -> wpc_symbols:Device_C; Link https://www.digikey.com/en/products/result?keywords=CL21B33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 -> https://search.kemet.com/download/specsheet/C0805C333K5RACTU; MPN CL21B333KBANNNC -> C0805C333K5RACTU; Manufacturer Samsung -> KEMET
- C37: symbol Device:C -> wpc_symbols:Device_C; Link https://www.digikey.com/en/products/result?keywords=CL21C47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 -> https://search.kemet.com/download/specsheet/C0805C471J5GACTU; MPN CL21C471JBANNNC -> C0805C471J5GACTU; Manufacturer Samsung -> KEMET
- C43: symbol Device:C -> wpc_symbols:Device_C; Link https://www.digikey.com/en/products/result?keywords=CL21C39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 -> https://search.kemet.com/download/specsheet/C0805C391J5GACTU; MPN CL21C391JBANNNC -> C0805C391J5GACTU; Manufacturer Samsung -> KEMET
- C5: value 10000uF 25V -> 10000uF 35V; footprint Capacitor_THT:CP_Radial_D25.0mm_P10.00mm_SnapIn -> Capacitor_THT:CP_Radial_D26.0mm_P10.00mm_SnapIn; symbol Device:C_Polarized -> wpc_symbols:Device_C_Polarized; Link https://www.digikey.com/en/products/detail/rubycon/25USC100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 -> https://product.tdk.com/en/search/capacitor/aluminum-electr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; MPN 25USC10000MEFCSN25X25 -> B41252A7109M000; Manufacturer Rubycon -> TDK; Price (none) -> 8.71; Price100 1.85 -> 4.66992
- D101, D102, D103, D104: value STPS20M100S -> STPS20M100ST; footprint wpc_cost:D2PAK_Schottky_AKA -> wpc_cost:TO220_Schottky_AKA_5772; symbol Device:D_Schottky -> wpc_symbols:Device_D_Schottky; Link https://www.digikey.com/en/products/detail/stmicroelectronics/STPS20M100SG-TR/2122461 -> https://www.digikey.com/en/products/detail/stmicroelectronics/STPS20M100ST/2122463; MPN STPS20M100SG-TR -> STPS20M100ST
- D105, D106, D107, D108, D109, D110, D111, D112, D113, D114, D115, D116, D36, D37: symbol Device:D_Schottky -> wpc_symbols:Device_D_Schottky
- F103, F104, F105, F111, F112, F113, F114, F115, F116: symbol Device:Fuse -> wpc_symbols:Device_Fuse
- H1, H2, H3, H4, H5, H6, H7, H8: symbol Mechanical:MountingHole -> wpc_symbols:Mechanical_MountingHole
- J101, J109, J114: symbol Connector_Generic:Conn_01x07 -> wpc_symbols:Connector_Generic_Conn_01x07; Link https://www.digikey.com/en/products/result?keywords=0026604007 -> https://www.digikey.com/en/products/result?keywords=0026604070; MPN 0026604007 -> 0026604070
- J102, J110: symbol Connector_Generic:Conn_01x09 -> wpc_symbols:Connector_Generic_Conn_01x09; MPN 0026604009 -> 0026604090
- J103, J116, J117, J118: symbol Connector_Generic:Conn_01x04 -> wpc_symbols:Connector_Generic_Conn_01x04; Link https://www.digikey.com/en/products/result?keywords=0026604004 -> https://www.digikey.com/en/products/result?keywords=0026604040; MPN 0026604004 -> 0026604040
- J104, J106, J112: symbol Connector_Generic:Conn_01x05 -> wpc_symbols:Connector_Generic_Conn_01x05; Link https://www.digikey.com/en/products/result?keywords=0026604005 -> https://www.digikey.com/en/products/result?keywords=0026604050; MPN 0026604005 -> 0026604050
- J107: symbol Connector_Generic:Conn_01x06 -> wpc_symbols:Connector_Generic_Conn_01x06; Link https://www.digikey.com/en/products/result?keywords=0026604006 -> https://www.digikey.com/en/products/result?keywords=0026604060; MPN 0026604006 -> 0026604060
- J108: symbol Connector_Generic:Conn_01x03 -> wpc_symbols:Connector_Generic_Conn_01x03; Link https://www.digikey.com/en/products/result?keywords=0026604003 -> https://www.digikey.com/en/products/result?keywords=0026604030; MPN 0026604003 -> 0026604030
- L1, L2: symbol Device:L -> wpc_symbols:Device_L
- LED1, LED2, LED4, LED5, LED6, LED7: symbol Device:LED -> wpc_symbols:Device_LED
- R192, R193, R194, R196, R250, R251, R259, R260, R261, R262, R263, R264, R265, R266, R267, R268, R269, R270, R271, R272: symbol Device:R -> wpc_symbols:Device_R
- TP1, TP2, TP3, TP5, TP6, TP7, TP8, TP9: symbol Connector:TestPoint -> wpc_symbols:Connector_TestPoint
- U20, U21: symbol Regulator_Switching:TPS54360DDA -> wpc_symbols:Regulator_Switching_TPS54360DDA
Other:
- note added: "BR1: D101-D104 STPS20M100ST TO-220, each with 577202B00000G heatsink (tabs/heatsinks = cathodes; do not join heatsinks)"
- note added: "Power supplies (windings per manual/pinwiki: 9 VAC red -> +5V, 13.3 VAC blu-wht -> +18V, 16 VAC wht-red -> +20V, 51 VAC blk-yel -> "+50V" (~70 V DC), 9.8 VAC wht-grn -> +12V power). Each secondary is fused (F111-F114, F116, 5x20 mm) before its bridge: GBPC3510W block (BR3, 6223BG basket heatsink); the +18V (D101-D104), BR1 D101-D104 use STPS20M100ST TO-220AB with individual 577202B00000G heatsink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"
- note removed: "BR1: discrete Schottky bridge D101-D104 (D2PAK tabs = cathodes: D101/D102 on the +18V pour, D103/D104 on the AC pours)"
- note removed: "Power supplies (windings per manual/pinwiki: 9 VAC red -> +5V, 13.3 VAC blu-wht -> +18V, 16 VAC wht-red -> +20V, 51 VAC blk-yel -> "+50V" (~70 V DC), 9.8 VAC wht-grn -> +12V power). Each secondary is fused (F111-F114, F116, 5x20 mm) before its bridge: GBPC3510W block (BR3, 6224BG basket heatsink); the +18V (D101-D104), +5V raw (D105-D108), +20V (D109-D112) and +12V power (D113-D116) bridges are f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"
