File: sol_highpower.kicad_sch (KiCad schematic)
At the start: 37 parts, among them J130 J130 Sol 1-8 drive (playfield), J131 J131 Sol 5-8 drive (cabinet, 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, J132 J132 Sol 1-4 drive (backbox, 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, Q64 IRLR3110ZTRPBF, Q66 IRLR3110ZTRPBF, Q68 IRLR3110ZTRPBF, Q70 IRLR3110ZTRPBF, Q76 IRLR3110ZTRPBF, Q78 IRLR3110ZTRPBF, Q80 IRLR3110ZTRPBF, Q82 IRLR3110ZTRPBF, U5 74HCT574

Commit message: Prepare WPC engineering candidate and verification tooling
Include revised PCB and schematics, component models, fabrication exports, renders, BOM, assembly counts, and reproducible electrical and manufacturing checks. Document unresolved replay convergence, regulator fault behavior, and physical qualification gates; this candidate is not production released.
Parts:
- B5: symbol Device:C -> wpc_symbols:Device_C
- D25, D26, D27, D28, D29, D30, D31, D32: symbol Diode:1N4007 -> wpc_symbols:Diode_1N4007
- J130: symbol Connector_Generic:Conn_01x09 -> wpc_symbols:Connector_Generic_Conn_01x09; MPN 0026604009 -> 0026604090
- J131, J132: symbol Connector_Generic:Conn_01x05 -> wpc_symbols:Connector_Generic_Conn_01x05; Link https://www.digikey.com/en/products/result?keywords=0026604005 -> https://www.digikey.com/en/products/result?keywords=0026604050; MPN 0026604005 -> 0026604050
- Q64, Q66, Q68, Q70, Q76, Q78, Q80, Q82: value IRLR3110ZTRPBF -> IPD90N10S4L06ATMA1; symbol Transistor_FET:Q_NMOS_GDS -> wpc_symbols:Transistor_FET_Q_NMOS_GDS; Link https://www.digikey.com/en/products/detail/infineon-technol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 -> https://www.infineon.com/part/IPD90N10S4L-06; MPN IRLR3110ZTRPBF -> IPD90N10S4L06ATMA1
- R126, R127, R128, R129, R130, R131, R132, R133, R134, R135, R136, R137, R138, R139, R140, R141: symbol Device:R -> wpc_symbols:Device_R
- U5: symbol 74xx:74HCT574 -> wpc_symbols:74xx_74HCT574
Other:
- note added: "High power solenoid drivers (sol. 1-8): IPD90N10S4L-06 DPAK (100 V, 14 mOhm, 16 mOhm at 4.5 V) driven directly by latch U5 (74HCT574, output HIGH = ON, outputs tri-stated by BLANKING -> gate pull-downs hold every driver OFF). SMC 3 A tie-back diodes return to +50V (the "+50V" rail of a WPC machine is ~70 V DC: 51 VAC winding, 72-78 V peak). U5 is clocked by /SOL 4 (J113-10). Output connectors J13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"
- note removed: "High power solenoid drivers (sol. 1-8): IRLR3110Z DPAK (100 V, 14 mOhm, 16 mOhm at 4.5 V) driven directly by latch U5 (74HCT574, output HIGH = ON, outputs tri-stated by BLANKING -> gate pull-downs hold every driver OFF). SMC 3 A tie-back diodes return to +50V (the "+50V" rail of a WPC machine is ~70 V DC: 51 VAC winding, 72-78 V peak). U5 is clocked by /SOL 4 (J113-10). Output connectors J130 (pl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"
- title: Solenoids 1-8 (high power, IRLR3110Z) -> Solenoids 1-8 (high power, IPD90N10S4L-06)
