File: sol_lowpower.kicad_sch (KiCad schematic)
At the start: 37 parts, among them J127 J127 Sol 9-16 drive (playfiel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, J128 J128 Sol 13-16 drive (cabinet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, J129 J129 Sol 9-12 drive (backbox,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, Q44 IRLR3110ZTRPBF, Q46 IRLR3110ZTRPBF, Q48 IRLR3110ZTRPBF, Q50 IRLR3110ZTRPBF, Q52 IRLR3110ZTRPBF, Q54 IRLR3110ZTRPBF, Q56 IRLR3110ZTRPBF, Q58 IRLR3110ZTRPBF, U4 74HCT574

Commit message: Prepare WPC engineering candidate and verification tooling
Include revised PCB and schematics, component models, fabrication exports, renders, BOM, assembly counts, and reproducible electrical and manufacturing checks. Document unresolved replay convergence, regulator fault behavior, and physical qualification gates; this candidate is not production released.
Parts:
- B4: symbol Device:C -> wpc_symbols:Device_C
- D17, D18, D19, D20, D21, D22, D23, D24: symbol Diode:1N4007 -> wpc_symbols:Diode_1N4007
- J127: symbol Connector_Generic:Conn_01x09 -> wpc_symbols:Connector_Generic_Conn_01x09; MPN 0026604009 -> 0026604090
- J128, J129: symbol Connector_Generic:Conn_01x05 -> wpc_symbols:Connector_Generic_Conn_01x05; Link https://www.digikey.com/en/products/result?keywords=0026604005 -> https://www.digikey.com/en/products/result?keywords=0026604050; MPN 0026604005 -> 0026604050
- Q44, Q46, Q48, Q50, Q52, Q54, Q56, Q58: value IRLR3110ZTRPBF -> IPD90N10S4L06ATMA1; symbol Transistor_FET:Q_NMOS_GDS -> wpc_symbols:Transistor_FET_Q_NMOS_GDS; Link https://www.digikey.com/en/products/detail/infineon-technol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 -> https://www.infineon.com/part/IPD90N10S4L-06; MPN IRLR3110ZTRPBF -> IPD90N10S4L06ATMA1
- R70, R71, R74, R75, R78, R79, R82, R83, R86, R87, R90, R91, R94, R95, R98, R99: symbol Device:R -> wpc_symbols:Device_R
- U4: symbol 74xx:74HCT574 -> wpc_symbols:74xx_74HCT574
Other:
- note added: "Low power solenoid drivers (sol. 9-16): IPD90N10S4L-06 logic-level DPAK MOSFETs (14 mOhm), latch U4 output HIGH = ON, clocked by /SOL 3 (J113-11). Tie-back diodes S3M (SMC, 3 A) to +50V (~70 V DC in the machine): coils in this group can be PWM-held by the firmware, the diode then carries the freewheel current. Output connectors J127 (playfield, key pin 2), J129 (backbox, sol 9-12, key 3) and J128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"
- note removed: "Low power solenoid drivers (sol. 9-16): IRLR3110Z logic-level DPAK MOSFETs (14 mOhm), latch U4 output HIGH = ON, clocked by /SOL 3 (J113-11). Tie-back diodes S3M (SMC, 3 A) to +50V (~70 V DC in the machine): coils in this group can be PWM-held by the firmware, the diode then carries the freewheel current. Output connectors J127 (playfield, key pin 2), J129 (backbox, sol 9-12, key 3) and J128 (cab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"
- title: Solenoids 9-16 (low power, IRLR3110Z) -> Solenoids 9-16 (low power, IPD90N10S4L-06)
