File: wpc_power_driver_cost.kicad_pcb (KiCad board)
At the start: 4 copper layers, 449.2 x 272.9 mm, 418 parts, among them J101 J101 xformer 9VAC (Red) / 13V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, J102 J102 xformer 16VAC (Wht-Red) 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, J103 J103 ground to 8-driver board, J104 J104 fused 51VAC (F112, pins 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, J105 J105 flipper AC (relay switch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, J106 J106 +20V to backbox flashlam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, J107 J107 +50V (F103/F104/F105) an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, J108 J108 spare (N/C), J109 J109 spare (N/C), J110 J110 spare (N/C), J111 J111 G.I. latch spare bits T5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, J112 J112 xformer 9.8VAC (Wht-Grn), J113 34-pin ribbon to CPU J211, J114 J114 +12V/+5V/GND to CPU J210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, J115 J115 G.I. 6.3VAC from transfo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, J116 J116 +12V power (unregulated)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, J117 J117 +12V power (unregulated)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, J118 J118 +12V power (unregulated)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, J119 J119 G.I. coin door (string 5), J120 J120 G.I. backbox (strings 2,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, J121 J121 G.I. playfield (strings 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, J122 J122 Sol 25-28 drive + tie-ba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, J123 J123 spare (N/C), J124 J124 Sol 25-28 drive (backbox), J125 J125 Sol 17-24 drive (backbox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, J126 J126 Sol 17-24 drive (playfie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, J127 J127 Sol 9-16 drive (playfiel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, J128 J128 Sol 13-16 drive (cabinet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, J129 J129 Sol 9-12 drive (backbox,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, J130 J130 Sol 1-8 drive (playfield), J131 J131 Sol 5-8 drive (cabinet, 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, J132 J132 Sol 1-4 drive (backbox, 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, J133 J133 lamp rows (cabinet), J134 J134 lamp rows (spare), J135 J135 lamp rows (playfield), J136 J136 lamp column 8 (cabinet), J137 J137 lamp columns (playfield), J138 J138 lamp columns (backbox), Q10 BTA16-600CRG, Q11 MMBT4401, Q12 BTA16-600CRG, Q13 MMBT4401, Q14 BTA16-600CRG, Q15 MMBT4401, Q16 BTA16-600CRG, Q17 MMBT4401, Q18 BTA16-600CRG, Q20 IRLR3110ZTRPBF, Q22 IRLR3110ZTRPBF, Q24 IRLR3110ZTRPBF, Q26 IRLR3110ZTRPBF, Q28 IRLR3110ZTRPBF, Q3 IRLR3110ZTRPBF (DNP), Q30 IRLR3110ZTRPBF, Q32 IRLR3110ZTRPBF, Q34 IRLR3110ZTRPBF, Q36 IRLR3110ZTRPBF, Q38 IRLR3110ZTRPBF, Q40 IRLR3110ZTRPBF, Q42 IRLR3110ZTRPBF, Q44 IRLR3110ZTRPBF, Q46 IRLR3110ZTRPBF, Q48 IRLR3110ZTRPBF, Q50 IRLR3110ZTRPBF, Q52 IRLR3110ZTRPBF, Q54 IRLR3110ZTRPBF, Q56 IRLR3110ZTRPBF, Q58 IRLR3110ZTRPBF, Q64 IRLR3110ZTRPBF, Q66 IRLR3110ZTRPBF, Q68 IRLR3110ZTRPBF, Q70 IRLR3110ZTRPBF, Q76 IRLR3110ZTRPBF, Q78 IRLR3110ZTRPBF, Q80 IRLR3110ZTRPBF, Q82 IRLR3110ZTRPBF, Q83 IRLR024NTRPBF, Q84 IRLR024NTRPBF, Q85 IRLR024NTRPBF, Q86 IRLR024NTRPBF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

Commit message: Prepare WPC engineering candidate and verification tooling
Include revised PCB and schematics, component models, fabrication exports, renders, BOM, assembly counts, and reproducible electrical and manufacturing checks. Document unresolved replay convergence, regulator fault behavior, and physical qualification gates; this candidate is not production released.
Parts:
- C11, C30, C5, C6, C7: value 10000uF 25V -> 10000uF 35V; footprint Capacitor_THT:CP_Radial_D25.0mm_P10.00mm_SnapIn -> Capacitor_THT:CP_Radial_D26.0mm_P10.00mm_SnapIn
- C21: footprint C_0805_2012Metric -> Capacitor_SMD:C_0805_2012Metric
- D101, D102, D103, D104: value STPS20M100SG -> STPS20M100ST; footprint D2PAK_Schottky_AKA -> wpc_cost:TO220_Schottky_AKA_5772
- D105, D106, D107, D108, D109, D110, D111, D112, D113, D114, D115, D116: value STPS20M100SG -> STPS20M100S; footprint D2PAK_Schottky_AKA -> wpc_cost:D2PAK_Schottky_AKA
- J103: value J103 ground to 8-driver board -> J103 ground to 8-driver board (all four pins grounded as on A-12697 sheet 1, no key)
- J105: value J105 flipper AC (relay switched, N/C on Fliptronic games) -> J105 fused 51VAC (F112, pins 1/2) and fused 16VAC (F111, pins 4/5) to the playfield - parallel to J104 as on A-12697 sh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
- J106: value J106 +20V to backbox flashlamps -> J106 +20V to backbox flashlamps (pins 1-4 open, key 4)
- J107: value J107 +50V (F103/F104/F105) and +20V to playfield -> J107 +50V (F103/F104/F105) and +20V (pins 5,6) to playfield
- J108: value J108 spare (N/C) -> J108 +50V (F103/F104/F105) to cabinet (N/C on STTNG)
- J113: footprint Connector_IDC:IDC-Header_2x17_P2.54mm_Vertical -> wpc_cost:3M_N2534_6002_RB
- J120: value J120 G.I. backbox (strings 2,3) -> J120 G.I. strings 1-5 (backbox harness uses strings 2,3)
- J121: value J121 G.I. playfield (strings 1,4,5) -> J121 G.I. strings 1-5 (playfield harness uses strings 1,4,5)
- J123: value J123 spare (N/C) -> J123 Sol 25-28 drive (backbox, parallel to J122/J124; N/C on STTNG)
- J126: value J126 Sol 17-24 drive (playfield flashers) -> J126 Sol 17-24 drive (playfield flashers) + tie-back cathodes of sol 21-24 on pins 10-13 (A-12697 D9-D12; N/C on STTNG)
- Q20, Q22, Q24, Q26, Q28, Q30, Q32, Q34, Q36, Q38, Q40, Q42, Q44, Q46, Q48, Q50, Q52, Q54, Q56, Q58, Q64, Q66, Q68, Q70, Q76, Q78, Q80, Q82: value IRLR3110ZTRPBF -> IPD90N10S4L06ATMA1
- Q3: value IRLR3110ZTRPBF (DNP) -> IPD90N10S4L06ATMA1
- R264: value 10.5K -> 11.3K
- R265: value 2K -> 2.1K
- moved D104 22.5 mm to (360.9, 17.6), turned to 0 degrees
- moved D102 22.3 mm to (378.5, 77.3), turned to 180 degrees
- moved D101 8.06 mm to (352.5, 53.4), turned to 180 degrees
- moved D103 7.78 mm to (347.5, 32.6), turned to 0 degrees
- moved C11 1.20 mm to (326.0, 16.5)
Routing:
- net AC13_B: track 165.2 -> 241.1 mm, vias 0 -> 6
- net D0: track 708.7 -> 675.4 mm
- net AC16_A: track 334.0 -> 353.5 mm, vias 5 -> 6
- net +18V: track 899.1 -> 908.2 mm, vias 31 -> 55
- net +5V: track 2324.6 -> 2315.6 mm, vias 59 -> 58
- net /Power_Supply/AC13_A_F: track 125.2 -> 128.6 mm, vias 2 -> 5
- net SOL06: track 194.2 -> 190.8 mm
- net D1: track 799.0 -> 801.8 mm
- net D7: track 713.1 -> 714.9 mm
- net D6_N: track 438.7 -> 440.6 mm
- net D5: track 818.5 -> 820.4 mm
- net D7_N: track 487.7 -> 489.3 mm
- net D3: track 787.9 -> 789.6 mm
- net D6: track 438.4 -> 439.8 mm
- net CLK_LAMP_ROW: track 591.9 -> 593.4 mm
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- added copper zone on In2.Cu, net +5V
Other:
- board text added: "CAUTION: UP TO 86 VDC"
- board text added: "J107 +50V/+20V"
- board text added: "J116 COIN DOOR"
- board text added: "J133 ROWS CAB"
- board text added: "J135 ROWS PF"
- board text added: "WPC A-12697-3 REV A"
- board text removed: "J107 +50V/+20V PLAYFIELD"
- board text removed: "J116 +12V/+5V COIN DOOR"
- board text removed: "J133 LAMP ROWS CAB"
- board text removed: "J135 LAMP ROWS PF"
